File: src/pcb/MCU.kicad_sch (KiCad schematic)
At the start: 6 parts, among them J1 Conn_01x05_Pin, J2 Conn_01x16_Pin, U3 74HC595, U4 74HC165, U5 74HC165

Commit message: Updated kicad schematic
Parts:
- U1: footprint Package_DIP:DIP-20_W7.62mm -> Package_DIP:DIP-20_W7.62mm_LongPads
- U3, U4, U5: footprint (none) -> Package_DIP:DIP-16_W7.62mm_LongPads
Changed lines of the file:
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@@
 			)
 		)
-		(property "Footprint" ""
+		(property "Footprint" "Package_DIP:DIP-16_W7.62mm_LongPads"
 			(at 78.74 86.36 0)
 			(effects
@@
 			)
 		)
-		(property "Footprint" ""
+		(property "Footprint" "Package_DIP:DIP-16_W7.62mm_LongPads"
 			(at 71.12 147.32 0)
 			(effects
@@
 			)
 		)
-		(property "Footprint" ""
+		(property "Footprint" "Package_DIP:DIP-16_W7.62mm_LongPads"
 			(at 121.92 152.4 0)
 			(effects
@@
 			)
 		)
-		(property "Footprint" "Package_DIP:DIP-20_W7.62mm"
+		(property "Footprint" "Package_DIP:DIP-20_W7.62mm_LongPads"
 			(at 153.67 48.26 0)
 			(effects
