File: src/pcb/rhythm.kicad_sch (KiCad schematic)
At the start: 0 parts

Commit message: Updated kicad schematic
Parts:
- added C10, C24: 0.47uF, symbol Device:C_Polarized_US
- added C11, C9: 47nF, symbol Device:C
- added C12, C13, C23: 0.1uF, symbol Device:C_Polarized_US
- added C14, C16, C18: 4.7nF, symbol Device:C
- added C15, C17: 1.5nF, symbol Device:C
- added C19, C21: 33nF, symbol Device:C
- added C20, C22: 10nF, symbol Device:C
- added C25: 0.15uF, symbol Device:C_Polarized_US
- added C26: 0.22uF, symbol Device:C_Polarized_US
- added C27: 15nF, symbol Device:C
- added C28, C30: 1nF, symbol Device:C
- added C29: 3.3nF, symbol Device:C
- added D10, D3, D4, D5, D6, D7, D8, D9: 1N4148, Diode_THT:D_DO-35_SOD27_P7.62mm_Horizontal, symbol Diode:1N4148
- added L1: 47mH, symbol Device:L
- added Q3: 2N3904, Package_TO_SOT_THT:TO-92_Inline, symbol Transistor_BJT:2N3904
- added R17: 100K, symbol Device:R_US
- added R18, R31, R40: 470K, symbol Device:R_Variable_US
- added R19, R20, R21, R30, R33, R39, R42: 68K, symbol Device:R_US
- added R22, R28, R37, R41: 330K, symbol Device:R_US
- added R23, R27, R36, R46, R50: 47K, symbol Device:R_US
- added R24, R26, R35, R38, R44, R45, R49, R53: 22K, symbol Device:R_US
- added R25, R47, R51: 220K, symbol Device:R_US
- added R29: 15K, symbol Device:R_US
- added R32, R43: 560K, symbol Device:R_US
- added R34, R48, R52: 470K, symbol Device:R_US
- added R54, R55, R56: 1M, symbol Device:R_US
- added RV1: 100K, symbol Device:R_Potentiometer_Trim_US
- added U8: 4011, Package_DIP:DIP-14_W7.62mm_LongPads, symbol 4xxx:4011
- added U9: ~, Package_DIP:DIP-8_W7.62mm_LongPads, symbol custom:PIC16F18313
Connections:
- new net: C9.1, R18.1, R20.2, U8.1, U8.2
- new net: C11.1, R17.1, R19.1, U8.3
- new net: R56.2, RV1.1
- new net: C30.1, RV1.2
- new net: C27.1, D8.1 (K), R52.2
- new net: C19.1, D6.1 (K), R35.1
- new net: C19.2, R36.1, R37.2
- new net: C22.1, R41.1, R42.1, U8.4
- new net: C20.2, C22.2, C23.1, D5.1 (K), R38.1
- new net: C10.1, R19.2, R20.1
- new net: R17.2, R18.2
- new net: C26.1, D10.1 (K), D9.1 (K), R49.1
- new net: D8.2 (A), R51.1
- new net: C26.2, R50.1, R51.2
- new net: C28.1, U9.3 (RA4)
- new net: C16.1, R30.1, R33.2
- new net: C17.1, R32.1, R33.1, U8.10
- new net: C23.2, R43.2
- new net: C15.2, C17.2, C18.1, D4.1 (K), R29.1
- new net: C24.2, R46.1, R47.2
- new net: C15.1, R30.2, R31.1, U8.8, U8.9
- new net: D5.2 (A), R37.1
- new net: C29.2, C30.2, L1.2, Q3.3 (C)
- new net: C28.2, R54.1
- new net: Q3.2 (B), R48.1, R52.1, R54.2, R55.1
- new net: C12.2, R22.2, R23.1
- new net: R31.2, R32.2
- new net: C25.1, D7.1 (K), R48.2
- new net: R40.2, R41.2
- new net: D7.2 (A), R47.1
- new net: C20.1, R39.2, R40.1, U8.5, U8.6
- new net: D3.2 (A), R22.1
- new net: D4.2 (A), R28.1
- new net: C14.2, R27.1, R28.2
- new net: C11.2, C13.1, C9.2, D3.1 (K), R21.1
- new net: C21.1, R39.1, R42.2
- new net: C13.2, R25.2
- new net: C18.2, R34.2
- new net +5V: C29.1, L1.1, U8.14 (VDD), U9.1 (Vdd)
- new net BD_TRIG: C12.1, R24.1
- new net CL_TRIG: C14.1, R26.1
- new net CY_TRIG: C24.1, R45.1
- new net GND: C10.2, C16.2, C21.2, C25.2, C27.2, Q3.1 (E), R21.2, R23.2, R24.2, R26.2, R27.2, R29.2, R35.2, R36.2, R38.2, R44.2, R45.2, R46.2, R49.2, R50.2, R53.2, R55.2, RV1.3, U8.12, U8.13, U8.7 (VSS), U9.8 (Vss)
- new net HH_TRIG: D9.2 (A), R53.1
- new net RHYTHM: R25.1, R34.1, R43.1, R56.1
- new net SD_TRIG: D10.2 (A), D6.2 (A), R44.1
